File: quickey/quickey.kicad_pcb (KiCad board)
At the start: 2 copper layers, 289.4 x 118 mm, 159 parts, among them J1 USB_C_Receptacle_USB2.0, SW1 SW_Push, U1 ATmega32U4-AU, Y1 Crystal_GND24_Small

Commit message: Pass DRC ERC
Parts:
- moved D68 12.7 mm to (271.3, 133.3), turned to 0 degrees
- moved H2 4.50 mm to (288.4, 132.2)
Routing:
- net ROW4: track 347.2 -> 332.9 mm, vias 22 -> 21
- net Net-(D68-Pad2): track 10.7 -> 18.8 mm
