File: quickey/quickey.sch (KiCad schematic (older format))
At the start: 18 parts

Commit message: Schematic and PCB
Parts:
- added D10, D11, D12, D13, D14, D15, D16, D17, D18, D19, D2, D20, D21, D22, D23, D24, D25, D26, D27, D28, D29, D3, D30, D31, D32, D33, D34, D35, D36, D37, D38, D39, D4, D40, D41, D42, D43, D44, D45, D46, D47, D48, D49, D5, D50, D51, D52, D53, D54, D55, D56, D57, D58, D59, D6, D60, D61, D62, D63, D64, D65, D66, D67, D68, D7, D8, D9: D_Small, Diode_SMD:D_SOD-123, symbol Device:D_Small
- added H1, H2, H3, H4, H5, H6, H7: MountingHole_Pad, MountingHole:MountingHole_2.2mm_M2_Pad, symbol Mechanical:MountingHole_Pad
- added Key_'1, Key_,1, Key_-1, Key_.1, Key_/1, Key_0, Key_1, Key_2, Key_3, Key_4, Key_5, Key_6, Key_7, Key_8, Key_9, Key_;1, Key_=1, Key_A1, Key_B1, Key_C1, Key_D1, Key_E1, Key_ESC1, Key_F1, Key_G1, Key_H1, Key_I1, Key_J1, Key_K1, Key_L1, Key_M1, Key_N1, Key_NEW1, Key_NEW2, Key_NEW3, Key_NEW4, Key_NEW5, Key_NEW6, Key_O1, Key_P1, Key_Q1, Key_R1, Key_S1, Key_T1, Key_U1, Key_V1, Key_W1, Key_X1, Key_Y1, Key_Z1, Key_[1, Key_}1: MX-NoLED, MX_Only:MXOnly-1U, symbol MX_Alps_Hybrid:MX-NoLED
- added Key_Bksp1: MX-NoLED, MX_Only:MXOnly-2U, symbol MX_Alps_Hybrid:MX-NoLED
- added Key_Caps1: MX-NoLED, MX_Only:MXOnly-1.75U, symbol MX_Alps_Hybrid:MX-NoLED
- added Key_Enter1, Key_LShift1: MX-NoLED, MX_Only:MXOnly-2.25U, symbol MX_Alps_Hybrid:MX-NoLED
- added Key_LAlt1, Key_LCtrl1, Key_LWin1, Key_RAlt1, Key_RCtrl1, Key_RMenu1, Key_RWin1: MX-NoLED, MX_Only:MXOnly-1.25U, symbol MX_Alps_Hybrid:MX-NoLED
- added Key_RShift1: MX-NoLED, MX_Only:MXOnly-2.75U, symbol MX_Alps_Hybrid:MX-NoLED
- added Key_Space1: MX-NoLED, MX_Only:MXOnly-6.25U, symbol MX_Alps_Hybrid:MX-NoLED
- added Key_Tab1, Key_|1: MX-NoLED, MX_Only:MXOnly-1.5U, symbol MX_Alps_Hybrid:MX-NoLED
- C1, C2, C3, C4, C5, C6: renamed from C?; footprint (none) -> Capacitor_SMD:C_0805_2012Metric
- C7: renamed from C?; value 0.1uF -> 10uF; footprint (none) -> Capacitor_SMD:C_0805_2012Metric
- F1: renamed from F?; footprint (none) -> Fuse:Fuse_1812_4532Metric
- J1: renamed from J?; footprint (none) -> Connector_USB:USB_C_Receptacle_HRO_TYPE-C-31-M-12
- R1, R2, R3, R4, R5: renamed from R?; footprint (none) -> Resistor_SMD:R_0805_2012Metric
- SW1: renamed from SW?; footprint (none) -> Button_Switch_SMD:SW_SPST_SKQG_WithoutStem
- Y1: renamed from Y?; footprint (none) -> Crystal:Crystal_SMD_3225-4Pin_3.2x2.5mm
- gave numbers to parts that had none: 2
Connections:
- net +5V: now also U1.14 (VCC), U1.2 (UVCC), U1.24 (AVCC), U1.34 (VCC), U1.44 (AVCC); no longer D1.4 (VCC)
- net GND: now also H1.1, H2.1, H3.1, H4.1, H5.1, H6.1, H7.1
- net VCC: now also D1.4 (VCC); no longer U1.14 (VCC), U1.2 (UVCC), U1.24 (AVCC), U1.34 (VCC), U1.44 (AVCC)
- net COL2: now reaches U1.10 (PB2)
- net COL2: now also Key_2.1 (COL), Key_LAlt1.1 (COL), Key_NEW1.1 (COL), Key_S1.1 (COL), Key_W1.1 (COL), Key_X1.1 (COL)
- net COL3: now reaches U1.11 (PB3)
- net COL3: now also Key_3.1 (COL), Key_C1.1 (COL), Key_D1.1 (COL), Key_E1.1 (COL), Key_NEW2.1 (COL)
- net COL4: now reaches U1.18 (PD0)
- net COL4: now also Key_4.1 (COL), Key_F1.1 (COL), Key_NEW3.1 (COL), Key_R1.1 (COL), Key_V1.1 (COL)
- net COL5: now reaches U1.19 (PD1)
- net COL5: now also Key_5.1 (COL), Key_B1.1 (COL), Key_G1.1 (COL), Key_NEW4.1 (COL), Key_Space1.1 (COL), Key_T1.1 (COL)
- net COL6: now reaches U1.20 (PD2)
- net COL6: now also Key_6.1 (COL), Key_H1.1 (COL), Key_N1.1 (COL), Key_NEW5.1 (COL), Key_Y1.1 (COL)
- net COL7: now reaches U1.21 (PD3)
- net COL7: now also Key_7.1 (COL), Key_J1.1 (COL), Key_M1.1 (COL), Key_NEW6.1 (COL), Key_U1.1 (COL)
- net COL8: now reaches U1.22 (PD5)
- net COL8: now also Key_,1.1 (COL), Key_8.1 (COL), Key_I1.1 (COL), Key_K1.1 (COL)
- net COL9: now reaches U1.28 (PB4)
- net COL9: now also Key_.1.1 (COL), Key_9.1 (COL), Key_L1.1 (COL), Key_O1.1 (COL)
- net COL10: now reaches U1.29 (PB5)
- net COL10: now also Key_/1.1 (COL), Key_0.1 (COL), Key_;1.1 (COL), Key_P1.1 (COL), Key_RAlt1.1 (COL)
- net COL11: now reaches U1.30 (PB6)
- net COL11: now also Key_'1.1 (COL), Key_-1.1 (COL), Key_RWin1.1 (COL), Key_[1.1 (COL)
- net COL12: now reaches U1.31 (PC6)
- net COL12: now also Key_=1.1 (COL), Key_RMenu1.1 (COL), Key_}1.1 (COL)
- net COL13: now reaches U1.32 (PC7)
- net COL13: now also Key_Bksp1.1 (COL), Key_Enter1.1 (COL), Key_RCtrl1.1 (COL), Key_RShift1.1 (COL), Key_|1.1 (COL)
- net ROW0: now reaches U1.36 (PF7)
- net ROW0: now also D12.1 (K), D18.1 (K), D2.1 (K), D23.1 (K), D28.1 (K), D34.1 (K), D39.1 (K), D44.1 (K), D48.1 (K), D52.1 (K), D57.1 (K), D61.1 (K), D64.1 (K), D7.1 (K)
- net ROW1: now reaches U1.37 (PF6)
- net ROW1: now also D13.1 (K), D19.1 (K), D24.1 (K), D29.1 (K), D3.1 (K), D35.1 (K), D40.1 (K), D45.1 (K), D49.1 (K), D53.1 (K), D58.1 (K), D62.1 (K), D65.1 (K), D8.1 (K)
- net ROW2: now reaches U1.38 (PF5)
- net ROW2: now also D14.1 (K), D20.1 (K), D25.1 (K), D30.1 (K), D36.1 (K), D4.1 (K), D41.1 (K), D46.1 (K), D50.1 (K), D54.1 (K), D59.1 (K), D66.1 (K), D9.1 (K)
- net ROW3: now reaches U1.39 (PF4)
- net ROW3: now also D10.1 (K), D15.1 (K), D21.1 (K), D26.1 (K), D31.1 (K), D37.1 (K), D42.1 (K), D47.1 (K), D5.1 (K), D51.1 (K), D55.1 (K), D67.1 (K)
- net ROW4: now reaches U1.40 (PF1)
- net ROW4: now also D11.1 (K), D16.1 (K), D32.1 (K), D56.1 (K), D6.1 (K), D60.1 (K), D63.1 (K), D68.1 (K)
- net ROW5: now reaches U1.41 (PF0)
- net ROW5: now also D17.1 (K), D22.1 (K), D27.1 (K), D33.1 (K), D38.1 (K), D43.1 (K)
- net COL0: now reaches U1.8 (PB0)
- net COL0: now also Key_Caps1.1 (COL), Key_ESC1.1 (COL), Key_LCtrl1.1 (COL), Key_LShift1.1 (COL), Key_Tab1.1 (COL)
- net COL1: now reaches U1.9 (PB1)
- net COL1: now also Key_1.1 (COL), Key_A1.1 (COL), Key_LWin1.1 (COL), Key_Q1.1 (COL), Key_Z1.1 (COL)
- new net: D4.2 (A), Key_Caps1.2 (ROW)
- new net: D9.2 (A), Key_A1.2 (ROW)
- new net: D14.2 (A), Key_S1.2 (ROW)
- new net: D20.2 (A), Key_D1.2 (ROW)
- new net: D25.2 (A), Key_F1.2 (ROW)
- new net: D30.2 (A), Key_G1.2 (ROW)
- new net: D36.2 (A), Key_H1.2 (ROW)
- new net: D41.2 (A), Key_J1.2 (ROW)
- new net: D46.2 (A), Key_K1.2 (ROW)
- new net: D50.2 (A), Key_L1.2 (ROW)
- new net: D54.2 (A), Key_;1.2 (ROW)
- new net: D59.2 (A), Key_'1.2 (ROW)
- new net: D66.2 (A), Key_Enter1.2 (ROW)
- new net: D5.2 (A), Key_LShift1.2 (ROW)
- new net: D10.2 (A), Key_Z1.2 (ROW)
- new net: D15.2 (A), Key_X1.2 (ROW)
- new net: D21.2 (A), Key_C1.2 (ROW)
- new net: D26.2 (A), Key_V1.2 (ROW)
- new net: D31.2 (A), Key_B1.2 (ROW)
- new net: D37.2 (A), Key_N1.2 (ROW)
- new net: D42.2 (A), Key_M1.2 (ROW)
- new net: D47.2 (A), Key_,1.2 (ROW)
- new net: D51.2 (A), Key_.1.2 (ROW)
- new net: D55.2 (A), Key_/1.2 (ROW)
- new net: D67.2 (A), Key_RShift1.2 (ROW)
- new net: D6.2 (A), Key_LCtrl1.2 (ROW)
- new net: D11.2 (A), Key_LWin1.2 (ROW)
- new net: D16.2 (A), Key_LAlt1.2 (ROW)
- new net: D32.2 (A), Key_Space1.2 (ROW)
- new net: D56.2 (A), Key_RAlt1.2 (ROW)
- new net: D60.2 (A), Key_RWin1.2 (ROW)
- new net: D63.2 (A), Key_RMenu1.2 (ROW)
- new net: D68.2 (A), Key_RCtrl1.2 (ROW)
- new net: D17.2 (A), Key_NEW1.2 (ROW)
- new net: D22.2 (A), Key_NEW2.2 (ROW)
- new net: D27.2 (A), Key_NEW3.2 (ROW)
- new net: D33.2 (A), Key_NEW4.2 (ROW)
- new net: D38.2 (A), Key_NEW5.2 (ROW)
- new net: D43.2 (A), Key_NEW6.2 (ROW)
- new net: D2.2 (A), Key_ESC1.2 (ROW)
- new net: D7.2 (A), Key_1.2 (ROW)
- new net: D12.2 (A), Key_2.2 (ROW)
- new net: D18.2 (A), Key_3.2 (ROW)
- new net: D23.2 (A), Key_4.2 (ROW)
- new net: D28.2 (A), Key_5.2 (ROW)
- new net: D34.2 (A), Key_6.2 (ROW)
- new net: D39.2 (A), Key_7.2 (ROW)
- new net: D44.2 (A), Key_8.2 (ROW)
- new net: D48.2 (A), Key_9.2 (ROW)
- new net: D52.2 (A), Key_0.2 (ROW)
- new net: D57.2 (A), Key_-1.2 (ROW)
- new net: D61.2 (A), Key_=1.2 (ROW)
- new net: D64.2 (A), Key_Bksp1.2 (ROW)
- new net: D3.2 (A), Key_Tab1.2 (ROW)
- new net: D8.2 (A), Key_Q1.2 (ROW)
- new net: D13.2 (A), Key_W1.2 (ROW)
- new net: D19.2 (A), Key_E1.2 (ROW)
- new net: D24.2 (A), Key_R1.2 (ROW)
- new net: D29.2 (A), Key_T1.2 (ROW)
- new net: D35.2 (A), Key_Y1.2 (ROW)
- new net: D40.2 (A), Key_U1.2 (ROW)
- new net: D45.2 (A), Key_I1.2 (ROW)
- new net: D49.2 (A), Key_O1.2 (ROW)
- new net: D53.2 (A), Key_P1.2 (ROW)
- new net: D58.2 (A), Key_[1.2 (ROW)
- new net: D62.2 (A), Key_}1.2 (ROW)
- new net: D65.2 (A), Key_|1.2 (ROW)

Commit message: Pass DRC ERC
Connections:
- no-connect marks 3 -> 9
Changed lines of the file:
@@
 Wire Wire Line
 	9300 6500 9300 6600
+NoConn ~ 2800 4800
+NoConn ~ 2800 5700
+NoConn ~ 2800 5900
+NoConn ~ 2800 6000
+NoConn ~ 2800 6200
+NoConn ~ 2800 6300
 $EndSCHEMATC
